File: Hardware/maskmoji.sch (KiCad schematic (older format))
At the start: 12 parts, among them J1 USB_B_Mini, J2 Conn_01x02, J3 Conn_01x22, Q1 PZT2222A, U1 CH330N, U2 BQ24075, U3 ESP32-WROOM-32, U4 LM1117-3.3

Commit message: add firmware dir
Connections:
- net labels added: MISO, MOSI, SCK, ~CS
- wire segments 36 -> 40
Other:
- note added: "Battery"
- note added: "Display FPC Connector"
Changed lines of the file:
@@
 encoding utf-8
 Sheet 1 1
-Title ""
-Date ""
-Rev ""
+Title "MaskMoji Schematic"
+Date "2020-09-18"
+Rev "0.1"
 Comp ""
 Comment1 ""
@@
 Text Label 3450 3000 1    50   ~ 0
 Backlight
+Wire Wire Line
+	4850 2650 4850 3500
+Wire Wire Line
+	4950 2650 4950 3500
+Wire Wire Line
+	5050 2650 5050 3500
+Wire Wire Line
+	5150 2650 5150 3500
+Text Label 4850 3300 1    50   ~ 0
+~CS
+Text Label 4950 3300 1    50   ~ 0
+SCK
+Text Label 5050 3300 1    50   ~ 0
+MOSI
+Text Label 5150 3300 1    50   ~ 0
+MISO
+Text Notes 9750 2050 1    50   ~ 0
+Display FPC Connector
+Text Notes 5450 6750 2    50   ~ 0
+Battery
 $EndSCHEMATC
